File: examples/nexdap-fresh/output/esp32c3_managed_rp2040_swd_coprocessor/01_01_power.kicad_sch (KiCad schematic)
At the start: 22 parts, among them J1 USB-C-16P

Commit message: Update NexDAP example outputs and fix KiCad mapping logic / 更新 NexDAP 示例输出并修正 KiCad 映射逻辑
Parts:
- removed ANT1: 2450AT18A100E, JLC-MCP:ANT-SMD_L3.2-W1.6, symbol JLC-MCP-Imported:2450AT18A100E
- removed C_RF_SHUNT1: 1.2pF, JLC-MCP:C0603, symbol JLC-MCP-Capacitors:CC0603KRX7R9BB104
- removed F1: MNCP380HSN05AAT1G, JLC-MCP:SOT-23-5_L3.0-W1.7-P0.95-LS2.8-BR, symbol JLC-MCP-Misc:MNCP380HSN05AAT1G
- removed L_RF1: 3.9nH, JLC-MCP:IND-SMD_L1.2-W0.7, symbol JLC-MCP-Imported:CS0402-3N9G-S
- removed R_BUCK_FB1: 100k, JLC-MCP:R0603, symbol JLC-MCP-Resistors:0603WAF1002T5E
- removed R_BUCK_FB2: 33k, JLC-MCP:R0603, symbol JLC-MCP-Resistors:0603WAF1002T5E
- added C_BUCK_IN_HF1, C_BUCK_OUT_HF1: 100nF, JLC-MCP:C0603, symbol JLC-MCP-Capacitors:CC0603KRX7R9BB104
- added D_VBUS_TVS1: SMF5.0A, JLC-MCP:SMF5.0A, symbol JLC-MCP-Diodes:SMBJ58A_C353350
- added F1: SMD1206-050-33, JLC-MCP:SMD1206-050-33, symbol JLC-MCP-Misc:POLYFUSE_2P
- added R_BUCK_FB1: 453k, JLC-MCP:R0603, symbol JLC-MCP-Resistors:0603WAF4533T5E
- added R_BUCK_FB2: 100k, JLC-MCP:R0603, symbol JLC-MCP-Resistors:0603WAF1003T5E
- C_BUCK_IN1, C_BULK_3V3: value 10uF -> 22uF
Connections:
- net +3V3_MAIN: now also C_BUCK_OUT_HF1.1, R_BUCK_FB1.1; no longer U_BUCK1.1 (EN)
- net +5V_USB_PROTECTED: now also U_BUCK1.1 (EN), C_BUCK_IN_HF1.1, F1.2
- net BUCK_FB: now also R_BUCK_FB1.2, R_BUCK_FB2.1
- net GND_HOST: now also C_BUCK_IN_HF1.2, C_BUCK_OUT_HF1.2, D_VBUS_TVS1.2, R_BUCK_FB2.2
- net USB_VBUS: now also D_VBUS_TVS1.1, F1.1
- no-connect marks 11 -> 8
