File: examples/nexdap-fresh/output/esp32c3_managed_rp2040_swd_coprocessor/02_02_mcu.kicad_sch (KiCad schematic)
At the start: 26 parts

Commit message: Update NexDAP example outputs and fix KiCad mapping logic / 更新 NexDAP 示例输出并修正 KiCad 映射逻辑
Parts:
- removed LED_DAP1: Blue, JLC-MCP:LED0603-RD, symbol JLC-MCP-Inductors:LTST-C191TBKT
- removed LED_PWR1: Green, JLC-MCP:LED0603-RD, symbol JLC-MCP-Inductors:LTST-C191TBKT
- removed LED_TGT1: Red, JLC-MCP:LED0603-RD, symbol JLC-MCP-Inductors:LTST-C191TBKT
- removed R_LED_DAP1, R_LED_TGT1: 330R, JLC-MCP:R0603, symbol JLC-MCP-Resistors:0603WAF1002T5E
- removed R_LED_PWR1: 330R, JLC-MCP:LED0603-RD, symbol JLC-MCP-Inductors:LTST-C191TBKT
- removed Y_ESP32: 40MHz, JLC-MCP:CRYSTAL-SMD_4P-L3.2-W2.5-BL, symbol JLC-MCP-Crystals:X322512MSB4SI
- added Y_ESP32: 40MHz, JLC-MCP:CRYSTAL-SMD_4P-L3.2-W2.5-BL, symbol JLC-MCP-Crystals:X322540MPB4SI
Connections:
- net +3V3_MAIN: now also U_RP2040.43 (ADC_AVDD)
- net ESP_RP_BOOTSEL_CTRL: now also U_ESP32.27 (U0RXD)
- net ESP_XTAL_N: now also Y_ESP32.2 (GND)
- net ESP_XTAL_P: now also Y_ESP32.1 (OSC1)
- net GND_HOST: now also U_RP2040.19 (TESTEN)
- net RP_TGT_SWCLK: now reaches U_RP2040.2 (GPIO0)
- net RP_TGT_SWDIO: now reaches U_RP2040.3 (GPIO1)
- net VTREF_ADC: now reaches U_RP2040.38 (GPIO26_ADC0)
- net TGT_SWO_IN: now reaches U_RP2040.7 (GPIO5)
- net RP_TGT_UART_TX: now reaches U_RP2040.8 (GPIO6)
- net RP_TGT_UART_RX: now reaches U_RP2040.9 (GPIO7)
- net ESP_TO_RP_IRQ: no longer names the net of U_RP2040.13 (GPIO10)
- net ESP_TO_RP_IRQ: no longer U_ESP32.27 (U0RXD)
- net HOST_SWO_IN: no longer names the net of U_RP2040.6 (GPIO4)
- no-connect marks 38 -> 32
