File: examples/nexdap-fresh/output/esp32c3_managed_rp2040_swd_coprocessor/03_03_target.kicad_sch (KiCad schematic)
At the start: 15 parts

Commit message: Update NexDAP example outputs and fix KiCad mapping logic / 更新 NexDAP 示例输出并修正 KiCad 映射逻辑
Parts:
- removed C_VTREF1: 0.1uF, JLC-MCP:C0603, symbol JLC-MCP-Capacitors:CC0603KRX7R9BB104
- removed D_TGT_ESD1: SRV05-4, JLC-MCP:SOT-23-6_L2.9-W1.6-P0.95-LS2.8-BL, symbol JLC-MCP-Diodes:SRV05-4_C2836319
- removed F_TGT1: 200mA, JLC-MCP:F0805, symbol JLC-MCP-Imported:0805L020_30XR
- removed JP_TGT_PWR1: 2P-Jumper, Connector_PinHeader_2.54mm:PinHeader_1x02_P2.54mm_Vertical, symbol Connector_Generic:Conn_01x02
- removed J_TGT1: Header-2.54-2x4P, JLC-MCP:HDR-TH_8P-P2.54-V-M-2X4, symbol JLC-MCP-Connectors:HDR-2X4-2.54
- removed Q_NRST1: 2N7002, JLC-MCP:SOT-23-3_L2.9-W1.3-P1.90-LS2.4-BR, symbol JLC-MCP-Transistors:2N7002
- removed R_NRST_PU1: 10k, JLC-MCP:R0603, symbol JLC-MCP-Resistors:0603WAF1002T5E
- removed R_SWCLK1, R_SWDIO1, R_SWO1, R_nRESET1: 22R, JLC-MCP:R0603, symbol JLC-MCP-Resistors:0603WAF1002T5E
- added C_VTREF: 0.1uF, JLC-MCP:C0603, symbol JLC-MCP-Capacitors:CC0603KRX7R9BB104
- added D_TGT_ESD: SRV05-4, JLC-MCP:SOT-23-6_L2.9-W1.6-P0.95-LS2.8-BL, symbol JLC-MCP-Diodes:SRV05-4_C2836319
- added F_TGT: 200mA, JLC-MCP:F0805, symbol JLC-MCP-Imported:0805L020_30XR
- added JP_TGT_PWR: 2P-Jumper, JLC-MCP:HDR-TH_2P-P2.54-V-M, symbol JLC-MCP-Connectors:HDR-1X2-2.54
- added J_TGT: Header-2.54-2x5P, JLC-MCP:HDR-TH_10P-P2.54-V-M-2X5, symbol JLC-MCP-Connectors:HDR-2X5-2.54
- added Q_NRST: 2N7002, JLC-MCP:SOT-23-3_L2.9-W1.3-P1.90-LS2.4-BR, symbol JLC-MCP-Transistors:2N7002
- added R_NRST_PU: 10k, JLC-MCP:R0603, symbol JLC-MCP-Resistors:0603WAF1002T5E
- added R_SWCLK, R_SWDIO, R_SWO, R_TGT_UART_RX, R_TGT_UART_TX, R_nRESET: 22R, JLC-MCP:R0603, symbol JLC-MCP-Resistors:0603WAF1002T5E
Connections:
- net +3V3_MAIN is gone; now on net VTREF_TARGET: R_VTREF_DIV1.1
- net +5V_SW_TGT: now also JP_TGT_PWR.2, J_TGT.9
- net +5V_USB_PROTECTED: now also F_TGT.1
- net GND_HOST: now also C_VTREF.2, D_TGT_ESD.2, J_TGT.10, J_TGT.6, Q_NRST.2 (S)
- net HOST_nRESET_CTRL: now also Q_NRST.1 (G)
- net TGT_SWCLK: now also D_TGT_ESD.3, J_TGT.3, R_SWCLK.2
- net TGT_SWDIO: now also D_TGT_ESD.1, J_TGT.2, R_SWDIO.2
- net TGT_SWO_OUT: now also D_TGT_ESD.6, J_TGT.4, R_SWO.2
- net TGT_nRESET: now also D_TGT_ESD.4, J_TGT.5, R_nRESET.2
- net TGT_nRESET_DRV: now also Q_NRST.3 (D), R_NRST_PU.2, R_nRESET.1
- net VTREF_TARGET: now also D_TGT_ESD.5, J_TGT.1, R_NRST_PU.1; no longer R_VTREF_DIV1.2, R_VTREF_DIV2.1
- new net +5V_TGT_FUSED: F_TGT.2, JP_TGT_PWR.1
- new net RP_TGT_SWCLK: R_SWCLK.1
- new net RP_TGT_SWDIO: R_SWDIO.1
- new net RP_TGT_UART_RX: R_TGT_UART_RX.2
- new net RP_TGT_UART_TX: R_TGT_UART_TX.1
- new net TGT_SWO_IN: R_SWO.1
- new net TGT_UART_RX: J_TGT.8, R_TGT_UART_RX.1
- new net TGT_UART_TX: J_TGT.7, R_TGT_UART_TX.2
- new net VTREF_ADC: C_VTREF.1, R_VTREF_DIV1.2, R_VTREF_DIV2.1
- no-connect marks 2 -> 0
