File: examples/h618-agentboard-v1/hardware/schematic/initial/h618_agentboard_v1_initial/h618_agentboard_v1_initial.kicad_pcb (KiCad board)
At the start: 2 copper layers, 48 parts, among them J1 USB-C 5V input, J2 MicroSD boot slot, J3 UART0 debug header, J4 26-pin expansion header, J5 Future RP2040 / ESP32-class c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, J6 RJ45 with magnetics, J7 USB-A host port 1, J8 USB-A host port 2, J9 Micro HDMI, SW1 RESET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

Commit message: feat(h618): consolidate schematic sheets / 整理原理图分页
将 H618 KiCad 原理图从大量小分图整理为 8 个可评审模块页，补充分图 profile 和回归测试，并同步 H618 文档、模型、example 工程与 where 进度。

Consolidate the H618 KiCad schematic into eight reviewable module sheets, add sheet grouping coverage, and sync the H618 model, docs, generated example project, and where progress.
Parts:
- added R10: 10k, R0603, F.Cu at (132.1, 799.6)
- added R11: 47k, R0603, F.Cu at (40.6, 394.6)
- added R12: 47k, R0603, F.Cu at (92.4, 394.6)
- added R13: 47k, R0603, F.Cu at (144.1, 394.6)
- added R14: 47k, R0603, F.Cu at (195.8, 394.6)
- added R15: 47k, R0603, F.Cu at (247.5, 394.6)
- added R9: 10k, R0603, F.Cu at (128.4, 793.6)
- moved TP10 224.0 mm to (79.2, 1209.5)
- moved TP2 224.0 mm to (79.2, 980.0)
- moved TP7 224.0 mm to (61.2, 1125.7)
- moved TP1 224.0 mm to (73.2, 952.0)
- moved TP5 224.0 mm to (49.2, 1069.8)
- moved TP6 224.0 mm to (55.2, 1097.7)
- moved TP9 224.0 mm to (73.2, 1181.5)
- moved TP4 224.0 mm to (43.2, 1041.8)
- moved TP8 224.0 mm to (67.2, 1153.6)
- moved J7 213.5 mm to (67.9, 875.8)
- moved TP3 188.2 mm to (85.2, 1007.9)
- moved J6 118.6 mm to (206.7, 799.6)
- moved J8 109.8 mm to (152.6, 875.8)
- moved J9 109.8 mm to (237.4, 875.8)
- moved C3 84.1 mm to (124.5, 673.3)
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Connections:
- U4 pad 3: +3V3 -> H618_SPI0_WP_N
- U4 pad 7: +3V3 -> H618_SPI0_HOLD_N
