File: examples/h618-agentboard-v1/hardware/schematic/initial/h618_agentboard_v1_initial/h618_agentboard_v1_initial.kicad_sch (KiCad schematic)
At the start: 0 parts

Commit message: feat(h618): consolidate schematic sheets / 整理原理图分页
将 H618 KiCad 原理图从大量小分图整理为 8 个可评审模块页，补充分图 profile 和回归测试，并同步 H618 文档、模型、example 工程与 where 进度。

Consolidate the H618 KiCad schematic into eight reviewable module sheets, add sheet grouping coverage, and sync the H618 model, docs, generated example project, and where progress.
Other:
- removed sheet coprocessor_reserve
- removed sheet ethernet_magjack
- removed sheet h618_1v8
- removed sheet h618_24mhz_xtal
- removed sheet h618_32k_xtal
- removed sheet h618_3v3
- removed sheet h618_core
- removed sheet h618_fel_boot_pullup
- removed sheet h618_fel_key
- removed sheet h618_gpio
- removed sheet h618_pmic_i2c_pullup_scl
- removed sheet h618_pmic_i2c_pullup_sda
- removed sheet h618_pmic_input
- removed sheet h618_pmic_pwron_pullup
- removed sheet h618_reset_key
- removed sheet h618_soc_bga
- removed sheet indicator
- removed sheet input
- removed sheet io
- removed sheet lpddr4_2gb_memory
- removed sheet micro_hdmi_output
- removed sheet micro_sd_boot_socket
- removed sheet pmic_axp313a
- removed sheet reset
- removed sheet rgmii_gigabit_phy
- removed sheet spi_nor_16mb_flash
- removed sheet test_point
- removed sheet usb2_hub
- removed sheet usb_c_cc1_sink_rd
- removed sheet usb_c_cc2_sink_rd
- removed sheet usb_host_port_1
- removed sheet usb_host_port_2
- removed sheet usb_type_c_power_input
- added sheet boot_storage (04_boot_storage.kicad_sch)
- added sheet debug_control (05_debug_control.kicad_sch)
- added sheet display_expansion (08_display_expansion.kicad_sch)
- added sheet memory_ddr (03_memory_ddr.kicad_sch)
- added sheet network (06_network.kicad_sch)
- added sheet power_entry_pmic (01_power_entry_pmic.kicad_sch)
- added sheet soc_boot_clock (02_soc_boot_clock.kicad_sch)
- added sheet usb (07_usb.kicad_sch)
