File: examples/esp32c3-minimal-system/output/esp32c3_minimal_system/02_mcu.kicad_sch (KiCad schematic)
At the start: 6 parts, among them SW1 SW-SMD_6x6, SW2 SW-SMD_6x6, U1 ESP32-C3FH4

Commit message: docs: refresh verified examples / 文档：刷新已验证示例
Parts:
- removed C5: 1uF, JLC-MCP:C0603, symbol JLC-MCP:C1592
- removed R2: 10K, JLC-MCP:R0603, symbol JLC-MCP:C15401
- added C5: 1uF, JLC-MCP:C0603, symbol JLC-MCP:CL10A105KO8NNNC
- added R2: 10K, JLC-MCP:R0603, symbol JLC-MCP:0603WAJ0103T5E
Connections:
- net +3V3: now also R2.1
- net EN: now also C5.1
- net GND: now also C5.2
- net IO9: now also R2.2
