File: examples/esp32c3-minimal-system/output/esp32c3_minimal_system/03_io.kicad_sch (KiCad schematic)
At the start: 3 parts, among them J2 UART-4P

Commit message: docs: refresh verified examples / 文档：刷新已验证示例
Parts:
- removed J2: UART-4P, JLC-MCP:HDR-TH_4P-P2.54-H-M-W10.4, symbol JLC-MCP:2.54-1_4P
- added J2: UART-4P, JLC-MCP:HDR-TH_4P-P2.54-H-M-W10.4, symbol JLC-MCP:2.54-1*4P反弯排针
Changed lines of the file:
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@@
   (symbol
     (lib_id "JLC-MCP:RC0603JR-071KL")
-    (at 50.8 127 0)
+    (at 111.76 50.8 0)
     (unit 1)
     (exclude_from_sim no)
@@
     (on_board yes)
     (dnp no)
-    (property "Reference" "R3" (at 50.8 121.92 0)
+    (property "Reference" "R3" (at 111.76 45.72 0)
       (effects (font (size 1.27 1.27)))
     )
-    (property "Value" "1K" (at 50.8 132.08 0)
+    (property "Value" "1K" (at 111.76 55.88 0)
       (effects (font (size 1.27 1.27)))
     )
-    (property "Footprint" "JLC-MCP:R0603" (at 50.8 127 0)
+    (property "Footprint" "JLC-MCP:R0603" (at 111.76 50.8 0)
       (hide yes)
       (effects (font (size 1.27 1.27)))
@@
     (instances
       (project "esp32c3_minimal_system"
-        (path "/c6454059-6594-497e-831c-288c877860e1"
+        (path "/f24a40fa-5098-47d7-b8b7-13fc4119a715"
           (reference "R3")
           (unit 1)
@@
   (symbol
     (lib_id "JLC-MCP:APHD1608LCGCK")
-    (at 50.8 154.94 0)
+    (at 111.76 78.74 0)
     (unit 1)
     (exclude_from_sim no)
@@
     (on_board yes)
     (dnp no)
-    (property "Reference" "D1" (at 50.8 149.86 0)
+    (property "Reference" "D1" (at 111.76 73.66 0)
       (effects (font (size 1.27 1.27)))
     )
-    (property "Value" "LED0603" (at 50.8 160.02 0)
+    (property "Value" "LED0603" (at 111.76 83.82 0)
       (effects (font (size 1.27 1.27)))
     )
-    (property "Footprint" "JLC-MCP:LED-SMD_L1.6-W0.8-RD_GREEN-1" (at 50.8 154.94 0)
+    (property "Footprint" "JLC-MCP:LED-SMD_L1.6-W0.8-RD_GREEN-1" (at 111.76 78.74 0)
       (hide yes)
       (effects (font (size 1.27 1.27)))
@@
     (instances
       (project "esp32c3_minimal_system"
-        (path "/c6454059-6594-497e-831c-288c877860e1"
+        (path "/f24a40fa-5098-47d7-b8b7-13fc4119a715"
           (reference "D1")
           (unit 1)
@@
   )
   (symbol
-    (lib_id "JLC-MCP:2.54-1_4P")
-    (at 208.28 50.8 0)
+    (lib_id "JLC-MCP:2.54-1*4P反弯排针")
+    (at 50.8 50.8 0)
     (unit 1)
     (exclude_from_sim no)
@@
     (on_board yes)
     (dnp no)
-    (property "Reference" "J2" (at 208.28 45.72 0)
+    (property "Reference" "J2" (at 50.8 45.72 0)
       (effects (font (size 1.27 1.27)))
     )
-    (property "Value" "UART-4P" (at 208.28 55.88 0)
+    (property "Value" "UART-4P" (at 50.8 55.88 0)
       (effects (font (size 1.27 1.27)))
     )
-    (property "Footprint" "JLC-MCP:HDR-TH_4P-P2.54-H-M-W10.4" (at 208.28 50.8 0)
+    (property "Footprint" "JLC-MCP:HDR-TH_4P-P2.54-H-M-W10.4" (at 50.8 50.8 0)
       (hide yes)
       (effects (font (size 1.27 1.27)))
@@
     (instances
       (project "esp32c3_minimal_system"
-        (path "/c6454059-6594-497e-831c-288c877860e1"
+        (path "/f24a40fa-5098-47d7-b8b7-13fc4119a715"
           (reference "J2")
           (unit 1)
@@
     )
   )
-  (wire (pts (xy 45.72 127) (xy 41.91 127))
+  (wire (pts (xy 106.68 50.8) (xy 102.87 50.8))
     (stroke (width 0) (type default))
   )
-  (global_label "LED" (shape bidirectional) (at 41.91 127 0)
+  (global_label "LED" (shape bidirectional) (at 102.87 50.8 0)
     (effects (font (size 1.27 1.27)) (justify right))
   )
-  (wire (pts (xy 55.88 127) (xy 59.69 127))
+  (wire (pts (xy 116.84 50.8) (xy 120.65 50.8))
     (stroke (width 0) (type default))
   )
-  (global_label "GND" (shape input) (at 59.69 127 0)
+  (global_label "GND" (shape input) (at 120.65 50.8 0)
     (effects (font (size 1.27 1.27)) (justify left))
   )
-  (wire (pts (xy 45.72 156.21) (xy 41.91 156.21))
+  (wire (pts (xy 106.68 80.01) (xy 102.87 80.01))
     (stroke (width 0) (type default))
   )
-  (global_label "+3V3" (shape input) (at 41.91 156.21 0)
+  (global_label "+3V3" (shape input) (at 102.87 80.01 0)
     (effects (font (size 1.27 1.27)) (justify right))
   )
-  (wire (pts (xy 55.88 156.21) (xy 59.69 156.21))
+  (wire (pts (xy 116.84 80.01) (xy 120.65 80.01))
     (stroke (width 0) (type default))
   )
-  (global_label "GND" (shape input) (at 59.69 156.21 0)
+  (global_label "GND" (shape input) (at 120.65 80.01 0)
     (effects (font (size 1.27 1.27)) (justify left))
   )
-  (wire (pts (xy 203.2 50.8) (xy 199.39 50.8))
+  (wire (pts (xy 46.99 46.99) (xy 43.18 46.99))
     (stroke (width 0) (type default))
   )
-  (global_label "+3V3" (shape input) (at 199.39 50.8 0)
+  (global_label "+3V3" (shape input) (at 43.18 46.99 0)
     (effects (font (size 1.27 1.27)) (justify right))
   )
-  (wire (pts (xy 213.36 50.8) (xy 217.17 50.8))
+  (wire (pts (xy 46.99 49.53) (xy 43.18 49.53))
     (stroke (width 0) (type default))
   )
-  (global_label "UART_TX" (shape bidirectional) (at 217.17 50.8 0)
-    (effects (font (size 1.27 1.27)) (justify left))
+  (global_label "UART_TX" (shape bidirectional) (at 43.18 49.53 0)
+    (effects (font (size 1.27 1.27)) (justify right))
+  )
+  (wire (pts (xy 46.99 52.07) (xy 43.18 52.07))
+    (stroke (width 0) (type default))
+  )
+  (global_label "UART_RX" (shape bidirectional) (at 43.18 52.07 0)
+    (effects (font (size 1.27 1.27)) (justify right))
+  )
+  (wire (pts (xy 46.99 54.61) (xy 43.18 54.61))
+    (stroke (width 0) (type default))
+  )
+  (global_label "GND" (shape input) (at 43.18 54.61 0)
+    (effects (font (size 1.27 1.27)) (justify right))
   )
   (sheet_instances
     (path "/" (page "1"))
-    (path "/6ba1db61-53e2-4496-809d-7d5332c09378" (page "2"))
-    (path "/b66f7af6-2bc6-459d-9261-43e27a46edcb" (page "3"))
-    (path "/c6454059-6594-497e-831c-288c877860e1" (page "4"))
+    (path "/be7a3b58-92fe-4a65-a699-f9d10f5b89d1" (page "2"))
+    (path "/02f1ebc9-e6c7-4388-b578-06adebacdf96" (page "3"))
+    (path "/f24a40fa-5098-47d7-b8b7-13fc4119a715" (page "4"))
   )
 )
