File: examples/esp32c3-minimal-system/output/esp32c3_minimal_system/esp32c3_minimal_system.kicad_pcb (KiCad board)
At the start: 2 copper layers, 17 parts, among them J1 USB-C16PIN, J2 UART-4P, SW1 SW-SMD_6x6, SW2 SW-SMD_6x6, U1 ESP32-C3FH4, U2 AMS1117-3.3

Commit message: docs: refresh verified examples / 文档：刷新已验证示例
Parts:
- moved D1 221.8 mm to (285.6, 148.2)
- moved R3 221.8 mm to (279.6, 120.3)
- moved C6 163.6 mm to (240.1, 190.5)
- moved C7 71.1 mm to (50.8, 272.7)
- moved R1 71.1 mm to (125.4, 272.7)
- moved C5 71.1 mm to (168.1, 190.5)
- moved R2 71.1 mm to (200.0, 272.7)
- moved U2 68.6 mm to (64.4, 190.5)
- moved J2 10.2 mm to (236.7, 120.3)
- moved C1 2.54 mm to (128.8, 38.1)
- moved C2 2.54 mm to (134.8, 66.0)
- moved C3 2.54 mm to (140.8, 94.0)
- moved U1 2.54 mm to (198.1, 38.1)
