File: examples/stm32f103-minimal-system/output/stm32f103_minimal_system/stm32f103_minimal_system.kicad_pcb (KiCad board)
At the start: 2 copper layers, 18 parts, among them J1 USB-C16PIN, J2 SWD-4P, SW1 SW-TH_6x6, U1 STM32F103C8T6, U2 AMS1117-3.3, Y1 8MHz

Commit message: docs: refresh verified examples / 文档：刷新已验证示例
Parts:
- C5: footprint C0603 -> C0805
- J2: footprint HDR-TH_4P-P2.54-V-M-1 -> HDR-TH_2P-P2.54-V-M
- R2: footprint SOT-223-3_L6.5-W3.4-P2.30-LS7.0-BR -> R0603
- SW1: value SW-TH_6x6 -> SW-SMD_6x6; footprint SW-SMD_TK-6580S-2 -> SW-SMD_K5-1617SA-02
- moved U1 205.2 mm to (68.6, 114.3)
- moved D1 160.7 mm to (157.9, 232.1)
- moved R2 160.7 mm to (77.3, 204.1)
- moved R3 160.7 mm to (151.9, 204.1)
- moved J2 127.2 mm to (180.3, 210.1)
- moved C9 119.4 mm to (253.3, 176.2)
- moved Y1 119.4 mm to (253.3, 114.3)
- moved C8 119.4 mm to (247.3, 148.2)
- moved R1 106.7 mm to (178.0, 120.3)
- moved SW1 106.7 mm to (166.0, 154.2)
- moved C1 22.9 mm to (231.4, 38.1)
- moved C2 22.9 mm to (237.4, 66.0)
- moved C3 22.9 mm to (243.4, 94.0)
- moved C5 17.8 mm to (175.7, 66.0)
- moved C6 17.8 mm to (181.7, 94.0)
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