File: examples/ai-memory-badge-v1/output/ai_memory_badge_v1/01_usb_and_charging.kicad_sch (KiCad schematic)
At the start: 11 parts, among them J1 KH-TYPE-C-16P USB-C USB2.0 re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, J2 JST PH 2P SMD battery connect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, U3 MCP73831 LiPo charger, U6 USB2.0 ESD protection

Commit message: feat: split schematic layout from PCB placement / 将原理图布局与PCB摆位分离
Connections:
- net USB_D_P is gone; now on net GND: R22.2
