File: examples/ai-memory-badge-v1/output/ai_memory_badge_v1/03_esp32s3_core.kicad_sch (KiCad schematic)
At the start: 10 parts, among them SW1 Reset tactile switch, SW2 BOOT tactile switch, U1 ESP32-S3R8 bare SoC

Commit message: feat: split schematic layout from PCB placement / 将原理图布局与PCB摆位分离
Connections:
- net ESP_EN is gone; now on net GND: C7.1, R4.2, SW1.1 (a), U1.4 (CHIP_PU)
- net SYS_3V3 is gone; now on net GND: C3.1, C4.1, C5.1, C6.1, R4.1, R5.1, U1.20 (VDD3P3_RTC), U1.29 (VDD_SPI), U1.3 (VDD3P3), U1.46 (VDD3P3_CPU), U1.56 (VDDA)
