File: examples/ai-memory-badge-v1/output/ai_memory_badge_v1/04_memory.kicad_sch (KiCad schematic)
At the start: 4 parts, among them U4 W25Q128JVSIQ 16MB SPI flash, U5 8MB PSRAM reserve, DNP

Commit message: feat: split schematic layout from PCB placement / 将原理图布局与PCB摆位分离
Connections:
- net SYS_3V3 is gone; now on net GND: C10.1, C11.1, U4.8 (VCC)
