File: examples/ai-memory-badge-v1/output/ai_memory_badge_v1/07_storage.kicad_sch (KiCad schematic)
At the start: 6 parts, among them J5 microSD socket push-push

Commit message: feat: split schematic layout from PCB placement / 将原理图布局与PCB摆位分离
Connections:
- net SD_CS is gone; now on net GND: J5.2 (CD/DAT3), R14.2
- net SYS_3V3 is gone; now on net GND: C17.1, J5.4 (VDD), R14.1, R15.1, R24.1, R25.1
