File: examples/ai-memory-badge-v1/output/ai_memory_badge_v1/09_security_reserve.kicad_sch (KiCad schematic)
At the start: 4 parts, among them U7 I2C secure element, DNP

Commit message: feat: split schematic layout from PCB placement / 将原理图布局与PCB摆位分离
Connections:
- net SYS_3V3 is gone; now on net GND: C18.1, R20.1, R21.1, U7.8 (VCC)
