File: examples/ai-memory-badge-v1/output/ai_memory_badge_v1/ai_memory_badge_v1.kicad_pcb (KiCad board)
At the start: 2 copper layers, 81 parts, among them J1 KH-TYPE-C-16P USB-C USB2.0 re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, J2 JST PH 2P SMD battery connect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, J3 U.FL/IPEX antenna connector, J4 UART debug 4P, J5 microSD socket push-push, M1 LCM0827A3038F 3V flat vibrati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, Q1 AO3400A NMOS low-side switch, SW1 Reset tactile switch, SW2 BOOT tactile switch, SW3 Mark tactile switch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

Commit message: feat: split schematic layout from PCB placement / 将原理图布局与PCB摆位分离
Parts:
- removed TP1, TP10, TP11, TP12, TP13, TP14, TP2, TP3, TP4, TP5, TP6, TP7, TP8, TP9: TP, TP-SMD_1P
- added R26: 0R, R0603, F.Cu at (138.6, 18.4)
Connections:
- D1 pad 1: GND -> (no net)
- D1 pad 2: SYS_3V3 -> (no net)
- D2 pad 1: SYS_3V3 -> (no net)
- D2 pad 2: GND -> (no net)
- J3 pad 2: GND -> (no net)
- J5 pad 4: SYS_3V3 -> (no net)
- J5 pad 6: GND -> (no net)
- MK1 pad 1: MIC_3V3 -> (no net)
- MK1 pad 2: I2S_BCLK -> (no net)
- MK1 pad 3: GND -> (no net)
- MK1 pad 4: MIC_LR_SEL_L -> (no net)
- MK1 pad 5: I2S_LRCLK -> (no net)
- MK1 pad 6: I2S_DIN -> (no net)
- MK2 pad 1: MIC_3V3 -> (no net)
- MK2 pad 2: I2S_BCLK -> (no net)
- MK2 pad 3: GND -> (no net)
- MK2 pad 4: MIC_LR_SEL_R -> (no net)
- MK2 pad 5: I2S_LRCLK -> (no net)
- MK2 pad 6: I2S_DIN -> (no net)
- Q1 pad 1: MOTOR_GATE -> (no net)
- Q1 pad 2: GND -> (no net)
- Q1 pad 3: MOTOR_LOW -> (no net)
- U1 pad 1: RF_IO -> (no net)
- U1 pad 10: I2C_SCL -> (no net)
- U1 pad 11: BTN_MARK -> (no net)
- U1 pad 12: SD_CD -> (no net)
- U1 pad 13: SD_CS -> (no net)
- U1 pad 14: SD_MISO -> (no net)
- U1 pad 15: SD_SCLK -> (no net)
- U1 pad 16: SD_MOSI -> (no net)
- U1 pad 17: I2S_BCLK -> (no net)
- U1 pad 18: I2S_LRCLK -> (no net)
- U1 pad 19: I2S_DIN -> (no net)
- U1 pad 20: SYS_3V3 -> (no net)
- U1 pad 23: SW_MUTE -> (no net)
- U1 pad 24: MOTOR_DRV -> (no net)
- U1 pad 25: USB_D_N -> (no net)
- U1 pad 26: USB_D_P -> (no net)
- U1 pad 27: I2C_SDA -> (no net)
- U1 pad 28: PSRAM_CS -> (no net)
- U1 pad 29: SYS_3V3 -> (no net)
- U1 pad 3: SYS_3V3 -> (no net)
- U1 pad 30: FLASH_D2 -> (no net)
- U1 pad 31: FLASH_D3 -> (no net)
- U1 pad 32: FLASH_CS -> (no net)
- U1 pad 33: FLASH_CLK -> (no net)
- U1 pad 34: FLASH_D0 -> (no net)
- U1 pad 35: FLASH_D1 -> (no net)
- U1 pad 4: ESP_EN -> (no net)
- U1 pad 46: SYS_3V3 -> (no net)
- U1 pad 49: UART0_TX -> (no net)
- U1 pad 5: ESP_BOOT -> (no net)
- U1 pad 50: UART0_RX -> (no net)
- U1 pad 53: XTAL_N -> (no net)
- U1 pad 54: XTAL_P -> (no net)
- U1 pad 56: SYS_3V3 -> (no net)
- U1 pad 57: GND -> (no net)
- U1 pad 6: VBAT_SENSE -> (no net)
- U1 pad 7: LED_POWER -> (no net)
- U1 pad 9: LED_RECORD -> (no net)
- U2 pad 1: BAT_P -> (no net)
- U2 pad 2: GND -> (no net)
- U2 pad 3: BAT_P -> (no net)
- U2 pad 5: SYS_3V3_REG -> (no net)
- U3 pad 1: CHG_STAT -> (no net)
- U3 pad 2: GND -> (no net)
- U3 pad 3: BAT_P -> (no net)
- U3 pad 4: USB_5V -> (no net)
- U3 pad 5: CHG_PROG -> (no net)
- U4 pad 2: FLASH_D0 -> (no net)
- U4 pad 3: FLASH_D2 -> (no net)
- U4 pad 4: GND -> (no net)
- U4 pad 5: FLASH_D1 -> (no net)
- U4 pad 6: FLASH_CLK -> (no net)
- U4 pad 7: FLASH_D3 -> (no net)
- U4 pad 8: SYS_3V3 -> (no net)
- U5 pad 1: PSRAM_CS -> (no net)
- U5 pad 4: GND -> (no net)
- U5 pad 8: SYS_3V3 -> (no net)
- U7 pad 4: GND -> (no net)
- U7 pad 5: I2C_SDA -> (no net)
- U7 pad 6: I2C_SCL -> (no net)
- U7 pad 8: SYS_3V3 -> (no net)
- Y1 pad 4: GND -> (no net)
