File: examples/ai-memory-badge-v1/output/ai_memory_badge_v1/ai_memory_badge_v1.kicad_sch (KiCad schematic)
At the start: 0 parts

Commit message: refactor(example): rebuild ai-memory-badge with all topology fixes and optimizations
Circuit fixes:
- LED D1/D2 drive circuit corrected (GPIO controls LED via resistor)
- Mute switch redesigned (SPDT COM directly controls U9.ON)
- SYS_3V3 + EPD_3V3 merged for Rev A (J6.7 direct power)
- Removed J4 UART debug header, SW6 mode button, R16/R32 unused

Design optimizations:
- D3: BAT54C flyback diode across vibration motor M1
- C22: 100nF filter cap on VBAT_SENSE ADC input
- R24/R25: DNP (microSD CMD/DAT0 pullups unused in SPI mode)
- R11: mic power link connected to SYS_3V3
- R27/R28: corrected pullup/pulldown connections
- C20.1/C21.1: removed from SYS_3V3 (was shorting NFC antenna)
- R31.2/R32.2: removed from GND (was shorting button signals)
- J6.7/J7.2: fixed cross-net shorts

BOM consolidation:
- All passives unified to 0603 (was 0603+0805)
- SW4/SW5 unified to SMD SPDT slide switch (MST-12D18G4)
- SW1/SW2 moved to internal test sheet (not user-exposed)

3D models:
- 33 footprint files corrected to ${KIPRJMOD} relative paths
- New 3D models for downloaded components

Co-Authored-By: Claude <noreply@anthropic.com>
Parts:
- added C1, C14, C17, C2, C3: 10uF, C0603, symbol JLC-MCP:CL10A106KP8NNNC
- added C15, C16, C18, C19, C22, C4, C5, C6: 100nF, C0603, symbol JLC-MCP:CL10B104KA8NNNC
- added C20, C21: DNP, C0402, symbol JLC-MCP:0402CG150J500NT
- added C7: 1uF, C0603, symbol JLC-MCP:CL10A105KO8NNNC
- added D1: LED0603 green, LED-SMD_L1.6-W0.8-RD_GREEN-1, symbol JLC-MCP:APHD1608LCGCK
- added D2: LED0603 red, LED-SMD_L1.6-W0.8-R-RD, symbol JLC-MCP:KT-0603R
- added D3: BAT54 Schottky flyback, SOT-23-3_L2.9-W1.3-P1.90-LS2.4-BR, symbol JLC-MCP:BAT54C_FLYBACK
- added J1: KH-TYPE-C-16P USB-C USB2.0 receptacle, USB-C-SMD_KH-TYPE-C-16P, symbol JLC-MCP:KH-TYPE-C-16P
- added J2: JST PH 2P SMD battery connector, CONN-SMD_P2.00_S2B-PH-SM4-TB-LF-SN, symbol JLC-MCP:S2B-PH-SM4-TB
- added J5: microSD socket push-push, TF-SMD_TF-001B, symbol JLC-MCP:TF-001B
- added J6: 2.13 inch black-white e-paper SPI connector, FPC-SMD_24P-P0.50-L6.1-W16.4, symbol JLC-MCP:EPD_SPI_CONN_10P
- added J7: NFC antenna coil pads / connector, SMD-2P, symbol JLC-MCP:NFC_ANT_2P
- added M1: LCM0827A3038F 3V flat vibration motor, VIBRATIONMOTOR-TH_LCM0827A3038F, symbol JLC-MCP:LCM0827A3038F
- added MK1: MSM261S3526Z0CM I2S MEMS microphone left, MIC-SMD_6P-L3.5-W2.7-P0.90-TR, symbol JLC-MCP:MSM261S3526Z0CM
- added MK2: MSM261S3526Z0CM I2S MEMS microphone right, MIC-SMD_6P-L3.5-W2.7-P0.90-TR, symbol JLC-MCP:MSM261S3526Z0CM
- added Q1: AO3400A NMOS low-side switch, SOT-23-3_L2.9-W1.3-P1.90-LS2.4-BR, symbol JLC-MCP:AO3400A
- added R1, R2: 5.1K, R0603, symbol JLC-MCP:0603WAF5101T5E
- added R11, R12, R13, R22, R23, R26: 0R, R0603, symbol JLC-MCP:0603WAF0000T5E
- added R14, R15, R16, R19, R20, R21, R24, R25, R27, R31, R32, R4, R5: 10K, R0603, symbol JLC-MCP:0603WAJ0103T5E
- added R17: 100R, R0603, symbol JLC-MCP:0603WAF1000T5E
- added R18, R28: 100K, R0603, symbol JLC-MCP:0603WAF1003T5E
- added R3: 2K, R0603, symbol JLC-MCP:0603WAF2001T5E
- added R6, R7: 1K, R0603, symbol JLC-MCP:RC0603JR-071KL
- added R8: 1M, R0603, symbol JLC-MCP:0603WAF1004T5E
- added R9: 330K, R0603, symbol JLC-MCP:0603WAF3303T5E
- added SW1: Reset tactile switch, SW-SMD_K5-1617SA-02, symbol JLC-MCP:K5-1617SA-02
- added SW2: BOOT tactile switch, SW-SMD_K5-1617SA-02, symbol JLC-MCP:K5-1617SA-02
- added SW3: Mark tactile switch, SW-SMD_K5-1617SA-02, symbol JLC-MCP:K5-1617SA-02
- added SW4: Mute SPDT slide switch, SW-SMD_MST-12D18G4-SPDT-SLIDE-SWITCH, symbol JLC-MCP:MST-12D18G4SPDTSLIDESWITCH
- added SW5: REC slide switch SPDT, SW-SMD_MST-12D18G4-SPDT-SLIDE-SWITCH, symbol JLC-MCP:MST-12D18G4SPDTSLIDESWITCH
- added SW6: MODE side tactile button, SW-SMD_8P-L6.7-W5.4-P1.27-LS8.4, symbol JLC-MCP:DSHP04TSGER
- added U1: ESP32-S3-WROOM-1-N8R8 module, WIRELM-SMD_ESP32-S3-WROOM-1, symbol JLC-MCP:ESP32-S3-WROOM-1
- added U10: TPS22918 SD_3V3 load switch, SOT-23-6_L2.9-W1.6-P0.95-LS2.8-BL, symbol JLC-MCP:TPS22918DBVR
- added U2: AP2112K-3.3 600mA LDO, SOT-25-5_L2.9-W1.6-P0.95-LS2.8-BL, symbol JLC-MCP:AP2112K-3.3TRG1
- added U3: BQ24074 LiPo charger with power-path, QFN-16_L3.0-W3.0-P0.50-TL-EP1.7, symbol JLC-MCP:BQ24074RGTR
- added U6: USB2.0 ESD protection, SOT-23-6_L2.9-W1.6-P0.95-LS2.8-BL, symbol JLC-MCP:USBLC6-2SC6
- added U7: I2C secure element, DNP, SOIC-8_L4.9-W3.9-P1.27-LS6.0-BL, symbol JLC-MCP:ATECC608A-SSHDA-T_C616024
- added U8: ST25DV04KC dynamic NFC tag, SO-8_L4.9-W3.9-P1.27-LS6.0-BL, symbol JLC-MCP:ST25DV04KC-IE8S3
- added U9: TPS22918 MIC_3V3 load switch, SOT-23-6_L2.9-W1.6-P0.95-LS2.8-BL, symbol JLC-MCP:TPS22918DBVR
Connections:
- new net BAT_P: J2.1, U3.2 (BAT)
- new net BTN_MARK: SW3.1 (a), U1.6 (IO6)
- new net CC1: J1.A5 (CC1), R1.1
- new net CC2: J1.B5 (CC2), R2.1
- new net CHG_PROG: R3.1
- new net CHG_STAT: R19.2
- new net EPD_BUSY: J6.6 (EPD_BUSY), U1.31 (IO38)
- new net EPD_CS: J6.3 (EPD_CS), U1.28 (IO35)
- new net EPD_DC: J6.4 (EPD_DC), U1.29 (IO36)
- new net EPD_MOSI: J6.2 (EPD_MOSI)
- new net EPD_PWR_EN: J6.9 (PWR_EN), U1.8 (IO15)
- new net EPD_RST: J6.5 (EPD_RST), U1.30 (IO37)
- new net EPD_SCLK: J6.1 (EPD_SCLK)
- new net ESP_BOOT: R5.2, SW2.1 (a), U1.27 (IO0)
- new net ESP_EN: C7.1, R4.2, SW1.1 (a), U1.3 (EN)
- new net GND: C1.2, C14.2, C15.2, C16.2, C17.2, C18.2, C2.2, C20.2, C21.2, C22.2, C3.2, C4.2, C5.2, C6.2, C7.2, J1.1 (EP), J1.2 (EP), J1.3 (EP), J1.4 (EP), J1.A1 (GND), J1.A12 (GND), J1.B1 (GND), J1.B12 (GND), J2.2, J5.10 (SHIELD), J5.12 (SW), J5.6 (VSS), J5.9 (SHIELD), J6.8 (GND), MK1.3 (GND), MK2.3 (GND), Q1.2 (S), R1.2, R12.2, R13.1, R18.2, R2.2, R28.1, R3.2, R9.2, SW1.2 (b), SW2.2 (b), SW3.2 (b), U1.1 (GND), U10.2 (GND), U2.2 (GND), U3.8 (VSS), U6.2, U7.4 (GND), U8.4 (VSS), U9.2 (GND)
- new net I2C_SCL: R21.2, U1.5 (IO5), U7.6 (SCL), U8.6 (SCL)
- new net I2C_SDA: R20.2, U1.23 (IO21), U7.5 (SDA), U8.5 (SDA)
- new net I2S_BCLK: MK1.2 (SCK), MK2.2 (SCK), U1.20 (IO12)
- new net I2S_DIN: MK1.6 (SD), MK2.6 (SD), U1.22 (IO14)
- new net I2S_LRCLK: MK1.5 (WS), MK2.5 (WS), U1.21 (IO13)
- new net LED_POWER: D1.1 (K), R6.1
- new net LED_POWER_DRV: R6.2, U1.38 (IO2)
- new net LED_RECORD: D2.2 (K), R7.1
- new net LED_RECORD_DRV: R7.2, U1.4 (IO4)
- new net MIC_3V3: C15.1, C16.1, MK1.1 (VDD), MK2.1 (VDD), R11.2
- new net MIC_LR_SEL_L: MK1.4 (L/R), R12.1
- new net MIC_LR_SEL_R: MK2.4 (L/R), R13.2
- new net MIC_PWR_EN: SW4.1, U1.10 (IO17), U9.3 (ON)
- new net MIC_PWR_NC: R27.2, SW4.2
- new net MODE_BTN: U1.33 (IO40)
- new net MOTOR_DRV: R17.1, U1.11 (IO18)
- new net MOTOR_GATE: Q1.1 (G), R17.2, R18.1
- new net MOTOR_LOW: C19.2, D3.1 (A), M1.2, Q1.3 (D)
- new net NFC_ANT1: C20.1, J7.1 (AC0), U8.2 (AC0)
- new net NFC_ANT2: C21.1, J7.2 (AC1), U8.3 (AC1)
- new net NFC_GPO: U1.34 (IO41), U8.7 (GPO)
- new net REC_BTN: SW5.1, U1.32 (IO39)
- new net REC_STATE_NC: R31.2, SW5.2
- new net SD_3V3: C17.1, J5.4 (VDD), R14.1, R15.1, R24.1, R25.1
- new net SD_CD: J5.11 (SW), R15.2, U1.7 (IO7)
- new net SD_CS: J5.2 (CD/DAT3), R14.2, U1.12 (IO8)
- new net SD_MISO: J5.7 (DAT0), R25.2, U1.17 (IO9)
- new net SD_MOSI: J5.3 (CMD), R24.2, U1.19 (IO11)
- new net SD_PWR_EN: R28.2, U1.9 (IO16), U10.3 (ON)
- new net SD_SCLK: J5.5 (CLK), U1.18 (IO10)
- new net SYS_3V3: C18.1, C19.1, C3.1, C4.1, C5.1, C6.1, D1.2 (A), D2.1 (A), D3.2 (K), J6.7 (3V3), M1.1, R11.1, R20.1, R21.1, R26.2, R27.1, R31.1, R4.1, R5.1, U1.2 (3V3), U7.8 (VCC), U8.8 (VCC)
- new net SYS_3V3_REG: C2.1, R26.1, U2.5 (VOUT)
- new net UART0_RX: U1.36 (RXD0)
- new net UART0_TX: U1.37 (TXD0)
- new net USB_5V: C14.1, J1.A4 (VBUS), J1.A9 (VBUS), J1.B4 (VBUS), J1.B9 (VBUS), R19.1, U3.13 (IN), U6.5
- new net USB_D_N: R23.2, U1.13 (IO19)
- new net USB_D_N_CONN: J1.A7 (DN1), J1.B7 (DN2), U6.3
- new net USB_D_N_ESD: R23.1, U6.4
- new net USB_D_P: R22.2, U1.14 (IO20)
- new net USB_D_P_CONN: J1.A6 (DP1), J1.B6 (DP2), U6.1
- new net USB_D_P_ESD: R22.1, U6.6
- new net VBAT_SENSE: C22.1, R8.2, R9.1, U1.39 (IO1)
- new net VSYS: C1.1, R8.1, U2.1 (VIN), U2.3 (EN), U3.10 (OUT)
- no-connect marks 0 -> 59
Other:
- removed sheet 01_usb_and_charging
- removed sheet 02_system_power
- removed sheet 03_esp32s3_core
- removed sheet 04_memory
- removed sheet 05_clock_and_rf
- removed sheet 06_audio_front_end
- removed sheet 07_storage
- removed sheet 08_user_interface
- removed sheet 09_security_reserve
- removed sheet 10_test_and_bringup
- note added: "01 USB AND CHARGING"
- note added: "02 SYSTEM POWER"
- note added: "03 ESP32S3 CORE"
- note added: "04 DISPLAY EPAPER"
- note added: "05 NFC DYNAMIC TAG"
- note added: "06 AUDIO FRONT END"
- note added: "07 STORAGE"
- note added: "08 USER INTERFACE"
- note added: "09 SECURITY RESERVE"
- note added: "10 TEST AND BRINGUP"
- note added: "UNGROUPED"

Commit message: feat(example): 重建 ai-memory-badge 输出项目, 添加交接文档和 ERC 报告
Rebuild ai-memory-badge output project, add handoff doc and ERC reports

- 重新生成 .kicad_pro/.kicad_sch/.kicad_pcb/.kicad_prl 全套 KiCad 文件
- 更新输出目录中的 JLC-MCP 符号库和封装库 (镜像 source/libraries/)
- 新增 ERC 验证报告 (erc.json + erc.summary.json)
- 新增 kicad-execution-plan.json 和 jlc-mcp-install-report.json
- 新增 AIAgent.pretty 自定义封装目录
- 新增 pipeline-events.jsonl / simulation-*.json 流水线产物
- 删除残留锁文件 ~ai_memory_badge_v1.kicad_pro.lck
- 添加 HANDOFF.md 项目交接文档 (硬件架构/BOM 统计/文件结构/已知问题/投板清单)

Co-Authored-By: Claude <noreply@anthropic.com>
Parts:
- removed C20, C21: DNP, C0402, symbol JLC-MCP:0402CG150J500NT
- removed R16, R24, R25, R32: 10K, R0603, symbol JLC-MCP:0603WAJ0103T5E
- removed SW6: MODE side tactile button, SW-SMD_8P-L6.7-W5.4-P1.27-LS8.4, symbol JLC-MCP:DSHP04TSGER
- removed U7: I2C secure element, DNP, SOIC-8_L4.9-W3.9-P1.27-LS6.0-BL, symbol JLC-MCP:ATECC608A-SSHDA-T_C616024
- J7: now left out of the parts list
- SW1: value Reset tactile switch -> Reset pushbutton
- SW2: value BOOT tactile switch -> BOOT pushbutton
Connections:
- net EPD_MOSI: now also U1.25 (IO48)
- net EPD_SCLK: now also U1.24 (IO47)
- no-connect marks 59 -> 54
Other:
- note removed: "01 USB AND CHARGING"
- note removed: "02 SYSTEM POWER"
- note removed: "03 ESP32S3 CORE"
- note removed: "04 DISPLAY EPAPER"
- note removed: "05 NFC DYNAMIC TAG"
- note removed: "06 AUDIO FRONT END"
- note removed: "07 STORAGE"
- note removed: "08 USER INTERFACE"
- note removed: "09 SECURITY RESERVE"
- note removed: "10 TEST AND BRINGUP"
